File: HTSORENOIDv1.kicad_sch (KiCad schematic)
At the start: 21 parts, among them J1 Conn_01x04, J2 Conn_01x04, U1 STM32F303K8Tx, U2 ADP3338AKCZ-3.3, U3 NJM78L12SU3

Commit message: update
Parts:
- added D10, D11, D12, D6, D7, D8, D9: LED, LED_SMD:LED_0603_1608Metric_Pad1.05x0.95mm_HandSolder, symbol Device:LED
- added J10, J11, J12, J13, J14, J3, J4, J5, J6, J7, J8, J9: Conn_01x02, Connector_JST:JST_XH_S2B-XH-A_1x02_P2.50mm_Horizontal, symbol Connector_Generic:Conn_01x02
- added J15: Conn_01x04, Connector_PinHeader_2.54mm:PinHeader_1x04_P2.54mm_Vertical, symbol Connector_Generic:Conn_01x04
- added Q1, Q10, Q2, Q3, Q4, Q5, Q6, Q7, Q8, Q9: AO3400A, Package_TO_SOT_SMD:SOT-23, symbol Transistor_FET:AO3400A
- added R10, R11, R12, R13, R14, R15, R16, R17, R18, R19, R20, R21, R22, R23, R24, R25, R26, R27, R28, R29, R30, R31, R32, R33, R34, R35, R36, R37, R38, R39, R40, R41, R5, R6, R7, R8, R9: R, Resistor_SMD:R_0603_1608Metric_Pad0.98x0.95mm_HandSolder, symbol Device:R
- added U10, U11, U12, U13, U4, U5, U6, U7, U8, U9: TLP291, Package_SO:SOIC-4_4.55x2.6mm_P1.27mm, symbol Isolator:TLP291
- C4, C5, C7: footprint (none) -> Capacitor_SMD:C_0603_1608Metric_Pad1.08x0.95mm_HandSolder
- C6: footprint (none) -> Capacitor_SMD:C_0805_2012Metric_Pad1.18x1.45mm_HandSolder
- U3: footprint (none) -> Package_TO_SOT_SMD:TO-252-2
Connections:
- net +24V: now also J10.1 (Pin_1), J11.1 (Pin_1), J12.1 (Pin_1), J13.1 (Pin_1), J14.1 (Pin_1), J3.1 (Pin_1), J4.1 (Pin_1), J5.1 (Pin_1), J6.1 (Pin_1), J7.1 (Pin_1), J8.1 (Pin_1), J9.1 (Pin_1)
- net +3.3V: now also U1.1 (VDD), U1.17 (VDD), U1.5 (VDDA), J15.4 (Pin_4)
- net +8V: now also U10.4, U11.4, U12.4, U13.4, U4.4, U5.4, U6.4, U7.4, U8.4, U9.4
- net GND: now also U1.16 (VSS), U1.32 (VSS), D10.1 (K), D11.1 (K), D12.1 (K), D6.1 (K), D7.1 (K), D8.1 (K), D9.1 (K), J15.2 (Pin_2), R10.2, R11.2, R12.2, R13.2, R14.2, R5.2, R6.2, R7.2, R8.2, R9.2, U10.2, U11.2, U12.2, U13.2, U4.2, U5.2, U6.2, U7.2, U8.2, U9.2
- net GNDPWR: now also Q1.2 (S), Q10.2 (S), Q2.2 (S), Q3.2 (S), Q4.2 (S), Q5.2 (S), Q6.2 (S), Q7.2 (S), Q8.2 (S), Q9.2 (S), R15.1, R16.1, R17.1, R18.1, R19.1, R20.1, R21.1, R22.1, R23.1, R24.1
- net LED1: now also R35.1
- net LED2: now also R36.1
- net LED3: now also R37.1
- net LED4: now also R38.1
- net LED5: now also R39.1
- net LED6: now also R40.1
- net LED7: now also R41.1
- net SN1: now also R5.1, U4.1
- net SN10: now also R14.1, U13.1
- net SN2: now also R6.1, U5.1
- net SN3: now also R7.1, U6.1
- net SN4: now also R8.1, U7.1
- net SN5: now also R9.1, U8.1
- net SN6: now also R10.1, U9.1
- net SN7: now also R11.1, U10.1
- net SN8: now also R12.1, U11.1
- net SN9: now also R13.1, U12.1
- net SW1: now also J13.2 (Pin_2)
- net SW2: now also J14.2 (Pin_2)
- net SYS_SWCLK: now also J15.1 (Pin_1)
- net SYS_SWDIO: now also J15.3 (Pin_3)
- new net: R19.2, R29.1, U8.3
- new net: Q5.1 (G), R29.2
- new net: D7.2 (A), R36.2
- new net: R16.2, R26.1, U5.3
- new net: Q2.1 (G), R26.2
- new net: R23.2, R33.1, U12.3
- new net: R24.2, R34.1, U13.3
- new net: Q10.1 (G), R34.2
- new net: R20.2, R30.1, U9.3
- new net: Q1.1 (G), R27.2
- new net: R18.2, R28.1, U7.3
- new net: Q4.1 (G), R28.2
- new net: D9.2 (A), R38.2
- new net: R21.2, R31.1, U10.3
- new net: Q7.1 (G), R31.2
- new net: D10.2 (A), R39.2
- new net: R15.2, R27.1, U4.3
- new net: D6.2 (A), R35.2
- new net: Q6.1 (G), R30.2
- new net: D12.2 (A), R41.2
- new net: Q8.1 (G), R32.2
- new net: R17.2, R25.1, U6.3
- new net: Q9.1 (G), R33.2
- new net: Q3.1 (G), R25.2
- new net: R22.2, R32.1, U11.3
- new net: D11.2 (A), R40.2
- new net: D8.2 (A), R37.2
- new net O1: J3.2 (Pin_2), Q1.3 (D)
- new net O10: J12.2 (Pin_2), Q10.3 (D)
- new net O2: J5.2 (Pin_2), Q2.3 (D)
- new net O3: J7.2 (Pin_2), Q3.3 (D)
- new net O4: J9.2 (Pin_2), Q4.3 (D)
- new net O5: J11.2 (Pin_2), Q5.3 (D)
- new net O6: J4.2 (Pin_2), Q6.3 (D)
- new net O7: J6.2 (Pin_2), Q7.3 (D)
- new net O8: J8.2 (Pin_2), Q8.3 (D)
- new net O9: J10.2 (Pin_2), Q9.3 (D)
Other:
- moved on the sheet: D2, D3, D4, D5, J1, J2, R1, R2, R3, R4, U1

Commit message: update
Parts:
- removed J4, J5: Conn_01x02, Connector_JST:JST_XH_S2B-XH-A_1x02_P2.50mm_Horizontal, symbol Connector_Generic:Conn_01x02
- removed Q1, Q2: AO3400A, Package_TO_SOT_SMD:SOT-23, symbol Transistor_FET:AO3400A
- removed R15, R16, R26, R27: R, Resistor_SMD:R_0603_1608Metric_Pad0.98x0.95mm_HandSolder, symbol Device:R
- removed U10, U11, U12, U13, U4, U5, U6, U7, U8, U9: TLP291, Package_SO:SOIC-4_4.55x2.6mm_P1.27mm, symbol Isolator:TLP291
- added C11: 4.7u, Capacitor_SMD:C_0603_1608Metric_Pad1.08x0.95mm_HandSolder, symbol Device:C
- added C12, C13, C9: 0.1u, Capacitor_SMD:C_0603_1608Metric_Pad1.08x0.95mm_HandSolder, symbol Device:C
- added H1, H2, H3, H4: MountingHole, MountingHole:MountingHole_3.2mm_M3, symbol Mechanical:MountingHole
- added IC1: TJA1441AT_0Z, 0-Myparts:SOIC127P600X175-8N, symbol 0-Myparts:TJA1441AT_0Z
- added J16: Conn_01x04, Connector_PinHeader_2.54mm:PinHeader_1x04_P2.54mm_Vertical, symbol Connector_Generic:Conn_01x04
- added J17, J18: Conn_01x01_Pin, 0-Myparts:ねじ端子(縦), symbol Connector:Conn_01x01_Pin
- added JP1: Jumper_2_Bridged, Connector_PinHeader_2.54mm:PinHeader_1x02_P2.54mm_Vertical, symbol Jumper:Jumper_2_Bridged
- added R42: 10k, Resistor_SMD:R_0603_1608Metric, symbol Device:R
- added R43: 120, Resistor_SMD:R_0603_1608Metric, symbol Device:R
- added SW1, SW2: SW_Push, 0-Myparts:TVAF06, symbol Switch:SW_Push
- added U4, U5: TLP291-4, Package_SO:SOIC-16_4.55x10.3mm_P1.27mm, symbol Isolator:TLP291-4
Connections:
- net O1 is gone; now on net O6: J3.2 (Pin_2)
- net +24V: now also C5.1, J17.1 (Pin_1); no longer J13.1 (Pin_1), J14.1 (Pin_1)
- net +3.3V: now also J13.1 (Pin_1), J14.1 (Pin_1), C11.1, C9.1, IC1.5 (VIO), J16.4 (Pin_4), SW2.2
- net +8V: now also U4.10, U4.12, U4.14, U4.16, U5.10, U5.12, U5.14, U5.16
- net CANH: now also IC1.7 (CANH), JP1.1 (A)
- net CANL: now also IC1.6 (CANL), R43.2
- net CAN_RX: now also IC1.4 (RXD)
- net CAN_TX: now also IC1.1 (TXD)
- net GND: now also C11.2, C12.2, C13.2, C9.2, IC1.2 (GND), IC1.8 (S), J16.2 (Pin_2), R42.2, SW1.1, U4.2, U4.4, U4.6, U4.8, U5.2, U5.4, U5.6, U5.8
- net GNDPWR: now also J18.1 (Pin_1)
- net SN10: now also U5.1
- net SN3: now also U4.7
- net SN4: now also U4.5
- net SN5: now also U4.3
- net SN6: now also U4.1
- net SN7: now also U5.7
- net SN8: now also U5.5
- net SN9: now also U5.3
- net SW1: now also R6.1, U1.15 (PB1); no longer U1.14 (PB0)
- net SW2: now also R5.1, U1.14 (PB0); no longer U1.15 (PB1)
- net USART1_RX: now also J16.3 (Pin_3)
- net USART1_TX: now also J16.1 (Pin_1)
- net VCC: now also C13.1, IC1.3 (VCC)
- net at R19.2, R29.1: now also U4.13
- net at R23.2, R33.1: now also U5.13
- net at R24.2, R34.1: now also U5.15
- net at R20.2, R30.1: now also U4.15
- net at R18.2, R28.1: now also U4.11
- net at R21.2, R31.1: now also U5.9
- net at R17.2, R25.1: now also U4.9
- net at R22.2, R32.1: now also U5.11
- net BOOT: now reaches U1.31 (BOOT0)
- net BOOT: now also R42.1, SW2.1
- net NRST: now reaches U1.4 (NRST)
- net NRST: now also C12.1, SW1.2
- net SN1: no longer names the net of U1.2 (PF0)
- net SN1: no longer R5.1
- net SN2: no longer names the net of U1.3 (PF1)
- net SN2: no longer R6.1
- new net: JP1.2 (B), R43.1
- no-connect marks 0 -> 2
Other:
- note added: "BOOTSW"
- note added: "CANトランシーバー"
- note added: "RSTSW"
- moved on the sheet: C2, C3, C4, C5, C6, C7, D1, D2, D3, D4, D5, J1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
