File: HTSORENOIDv1.kicad_pcb (KiCad board)
At the start: 2 copper layers, 90 x 55 mm, 8 parts, among them J1 Conn_01x01_Pin, J2 Conn_01x01_Pin

Commit message: update
Parts:
- added C1: 1000u, Capacitor_THT:CP_Radial_D10.0mm_P5.00mm, F.Cu at (58.1, 105.7)
- added C2: 1u, Capacitor_SMD:C_0603_1608Metric_Pad1.08x0.95mm_HandSolder, F.Cu at (18.9, 100.3)
- added C3: 1u, Capacitor_SMD:C_0603_1608Metric_Pad1.08x0.95mm_HandSolder, F.Cu at (18.9, 102.8)
- added C4: 1u, Capacitor_SMD:C_0603_1608Metric_Pad1.08x0.95mm_HandSolder, F.Cu at (18.9, 105.3)
- added C5: 0.1u, Capacitor_SMD:C_0603_1608Metric_Pad1.08x0.95mm_HandSolder, F.Cu at (18.9, 107.8)
- added C6: 10u, Capacitor_SMD:C_0805_2012Metric_Pad1.18x1.45mm_HandSolder, F.Cu at (75.3, 97.0)
- added C7: 0.1u, Capacitor_SMD:C_0603_1608Metric_Pad1.08x0.95mm_HandSolder, F.Cu at (18.9, 110.3)
- added D10: LED, LED_SMD:LED_0603_1608Metric_Pad1.05x0.95mm_HandSolder, F.Cu at (50.5, 110.7)
- added D11: LED, LED_SMD:LED_0603_1608Metric_Pad1.05x0.95mm_HandSolder, F.Cu at (50.5, 113.3)
- added D12: LED, LED_SMD:LED_0603_1608Metric_Pad1.05x0.95mm_HandSolder, F.Cu at (50.5, 115.9)
- added D2: Blue, LED_SMD:LED_0603_1608Metric, F.Cu at (70.9, 86.8)
- added D3: Blue, LED_SMD:LED_0603_1608Metric, F.Cu at (70.9, 89.4)
- added D4: Blue, LED_SMD:LED_0603_1608Metric, F.Cu at (70.9, 92.0)
- added D5: Blue, LED_SMD:LED_0603_1608Metric, F.Cu at (70.9, 94.5)
- added D6: LED, LED_SMD:LED_0603_1608Metric_Pad1.05x0.95mm_HandSolder, F.Cu at (50.5, 100.3)
- added D7: LED, LED_SMD:LED_0603_1608Metric_Pad1.05x0.95mm_HandSolder, F.Cu at (50.5, 102.9)
- added D8: LED, LED_SMD:LED_0603_1608Metric_Pad1.05x0.95mm_HandSolder, F.Cu at (50.5, 105.5)
- added D9: LED, LED_SMD:LED_0603_1608Metric_Pad1.05x0.95mm_HandSolder, F.Cu at (50.5, 108.1)
- added J1: Conn_01x04, Connector_JST:JST_XH_S4B-XH-A_1x04_P2.50mm_Horizontal, F.Cu at (164.5, 82.7)
- added J10: Conn_01x02, Connector_JST:JST_XH_S2B-XH-A_1x02_P2.50mm_Horizontal, F.Cu at (48.6, 75.3)
- added J11: Conn_01x02, Connector_JST:JST_XH_S2B-XH-A_1x02_P2.50mm_Horizontal, F.Cu at (20.2, 88.8)
- added J12: Conn_01x02, Connector_JST:JST_XH_S2B-XH-A_1x02_P2.50mm_Horizontal, F.Cu at (29.7, 88.8)
- added J13: Conn_01x02, Connector_JST:JST_XH_S2B-XH-A_1x02_P2.50mm_Horizontal, F.Cu at (39.1, 88.8)
- added J14: Conn_01x02, Connector_JST:JST_XH_S2B-XH-A_1x02_P2.50mm_Horizontal, F.Cu at (48.6, 88.8)
- added J15: Conn_01x04, Connector_PinHeader_2.54mm:PinHeader_1x04_P2.54mm_Vertical, F.Cu at (66.5, 87.8)
- added J2: Conn_01x04, Connector_JST:JST_XH_S4B-XH-A_1x04_P2.50mm_Horizontal, F.Cu at (178.0, 82.7)
- added J3: Conn_01x02, Connector_JST:JST_XH_S2B-XH-A_1x02_P2.50mm_Horizontal, F.Cu at (20.2, 61.7)
- added J4: Conn_01x02, Connector_JST:JST_XH_S2B-XH-A_1x02_P2.50mm_Horizontal, F.Cu at (29.7, 61.7)
- added J5: Conn_01x02, Connector_JST:JST_XH_S2B-XH-A_1x02_P2.50mm_Horizontal, F.Cu at (39.1, 61.7)
- added J6: Conn_01x02, Connector_JST:JST_XH_S2B-XH-A_1x02_P2.50mm_Horizontal, F.Cu at (48.6, 61.7)
- added J7: Conn_01x02, Connector_JST:JST_XH_S2B-XH-A_1x02_P2.50mm_Horizontal, F.Cu at (20.2, 75.3)
- added J8: Conn_01x02, Connector_JST:JST_XH_S2B-XH-A_1x02_P2.50mm_Horizontal, F.Cu at (29.7, 75.3)
- added J9: Conn_01x02, Connector_JST:JST_XH_S2B-XH-A_1x02_P2.50mm_Horizontal, F.Cu at (39.1, 75.3)
- added Q1: AO3400A, Package_TO_SOT_SMD:SOT-23, F.Cu at (40.9, 101.3)
- added Q10: AO3400A, Package_TO_SOT_SMD:SOT-23, F.Cu at (45.8, 119.1)
- added Q2: AO3400A, Package_TO_SOT_SMD:SOT-23, F.Cu at (40.9, 105.7)
- added Q3: AO3400A, Package_TO_SOT_SMD:SOT-23, F.Cu at (40.9, 110.2)
- added Q4: AO3400A, Package_TO_SOT_SMD:SOT-23, F.Cu at (40.9, 114.6)
- added Q5: AO3400A, Package_TO_SOT_SMD:SOT-23, F.Cu at (40.9, 119.1)
- added Q6: AO3400A, Package_TO_SOT_SMD:SOT-23, F.Cu at (45.8, 101.3)
- added Q7: AO3400A, Package_TO_SOT_SMD:SOT-23, F.Cu at (45.8, 105.7)
- added Q8: AO3400A, Package_TO_SOT_SMD:SOT-23, F.Cu at (45.8, 110.2)
- added Q9: AO3400A, Package_TO_SOT_SMD:SOT-23, F.Cu at (45.8, 114.6)
- added R1: 10k, Resistor_SMD:R_0603_1608Metric, F.Cu at (74.9, 86.7)
- added R10: R, Resistor_SMD:R_0603_1608Metric_Pad0.98x0.95mm_HandSolder, F.Cu at (23.3, 102.8)
- added R11: R, Resistor_SMD:R_0603_1608Metric_Pad0.98x0.95mm_HandSolder, F.Cu at (23.3, 105.3)
- added R12: R, Resistor_SMD:R_0603_1608Metric_Pad0.98x0.95mm_HandSolder, F.Cu at (23.3, 107.8)
- added R13: R, Resistor_SMD:R_0603_1608Metric_Pad0.98x0.95mm_HandSolder, F.Cu at (23.3, 110.3)
- added R14: R, Resistor_SMD:R_0603_1608Metric_Pad0.98x0.95mm_HandSolder, F.Cu at (23.3, 112.8)
- added R15: R, Resistor_SMD:R_0603_1608Metric_Pad0.98x0.95mm_HandSolder, F.Cu at (23.3, 115.3)
- added R16: R, Resistor_SMD:R_0603_1608Metric_Pad0.98x0.95mm_HandSolder, F.Cu at (23.3, 117.9)
- added R17: R, Resistor_SMD:R_0603_1608Metric_Pad0.98x0.95mm_HandSolder, F.Cu at (23.3, 120.4)
- added R18: R, Resistor_SMD:R_0603_1608Metric_Pad0.98x0.95mm_HandSolder, F.Cu at (27.6, 100.3)
- added R19: R, Resistor_SMD:R_0603_1608Metric_Pad0.98x0.95mm_HandSolder, F.Cu at (27.6, 102.8)
- added R2: 10k, Resistor_SMD:R_0603_1608Metric, F.Cu at (74.9, 89.2)
- added R20: R, Resistor_SMD:R_0603_1608Metric_Pad0.98x0.95mm_HandSolder, F.Cu at (27.6, 105.3)
- added R21: R, Resistor_SMD:R_0603_1608Metric_Pad0.98x0.95mm_HandSolder, F.Cu at (27.6, 107.8)
- added R22: R, Resistor_SMD:R_0603_1608Metric_Pad0.98x0.95mm_HandSolder, F.Cu at (27.6, 110.3)
- added R23: R, Resistor_SMD:R_0603_1608Metric_Pad0.98x0.95mm_HandSolder, F.Cu at (27.6, 112.8)
- added R24: R, Resistor_SMD:R_0603_1608Metric_Pad0.98x0.95mm_HandSolder, F.Cu at (27.6, 115.3)
- added R25: R, Resistor_SMD:R_0603_1608Metric_Pad0.98x0.95mm_HandSolder, F.Cu at (27.6, 117.9)
- added R26: R, Resistor_SMD:R_0603_1608Metric_Pad0.98x0.95mm_HandSolder, F.Cu at (27.6, 120.4)
- added R27: R, Resistor_SMD:R_0603_1608Metric_Pad0.98x0.95mm_HandSolder, F.Cu at (32.0, 100.3)
- added R28: R, Resistor_SMD:R_0603_1608Metric_Pad0.98x0.95mm_HandSolder, F.Cu at (32.0, 102.8)
- added R29: R, Resistor_SMD:R_0603_1608Metric_Pad0.98x0.95mm_HandSolder, F.Cu at (32.0, 105.3)
- added R3: 1k, Resistor_SMD:R_0603_1608Metric, F.Cu at (74.9, 91.8)
- added R30: R, Resistor_SMD:R_0603_1608Metric_Pad0.98x0.95mm_HandSolder, F.Cu at (32.0, 107.8)
- added R31: R, Resistor_SMD:R_0603_1608Metric_Pad0.98x0.95mm_HandSolder, F.Cu at (32.0, 110.3)
- added R32: R, Resistor_SMD:R_0603_1608Metric_Pad0.98x0.95mm_HandSolder, F.Cu at (32.0, 112.8)
- added R33: R, Resistor_SMD:R_0603_1608Metric_Pad0.98x0.95mm_HandSolder, F.Cu at (32.0, 115.3)
- added R34: R, Resistor_SMD:R_0603_1608Metric_Pad0.98x0.95mm_HandSolder, F.Cu at (32.0, 117.9)
- added R35: R, Resistor_SMD:R_0603_1608Metric_Pad0.98x0.95mm_HandSolder, F.Cu at (32.0, 120.4)
- added R36: R, Resistor_SMD:R_0603_1608Metric_Pad0.98x0.95mm_HandSolder, F.Cu at (36.3, 100.3)
- added R37: R, Resistor_SMD:R_0603_1608Metric_Pad0.98x0.95mm_HandSolder, F.Cu at (36.3, 102.8)
- added R38: R, Resistor_SMD:R_0603_1608Metric_Pad0.98x0.95mm_HandSolder, F.Cu at (36.3, 105.3)
- added R39: R, Resistor_SMD:R_0603_1608Metric_Pad0.98x0.95mm_HandSolder, F.Cu at (36.3, 107.8)
- added R4: 10k, Resistor_SMD:R_0603_1608Metric, F.Cu at (74.9, 94.3)
- added R40: R, Resistor_SMD:R_0603_1608Metric_Pad0.98x0.95mm_HandSolder, F.Cu at (36.3, 110.3)
- added R41: R, Resistor_SMD:R_0603_1608Metric_Pad0.98x0.95mm_HandSolder, F.Cu at (36.3, 112.8)
- added R5: R, Resistor_SMD:R_0603_1608Metric_Pad0.98x0.95mm_HandSolder, F.Cu at (18.9, 112.8)
- added R6: R, Resistor_SMD:R_0603_1608Metric_Pad0.98x0.95mm_HandSolder, F.Cu at (18.9, 115.3)
- added R7: R, Resistor_SMD:R_0603_1608Metric_Pad0.98x0.95mm_HandSolder, F.Cu at (18.9, 117.9)
- added R8: R, Resistor_SMD:R_0603_1608Metric_Pad0.98x0.95mm_HandSolder, F.Cu at (18.9, 120.4)
- added R9: R, Resistor_SMD:R_0603_1608Metric_Pad0.98x0.95mm_HandSolder, F.Cu at (23.3, 100.3)
- added U1: STM32F303K8Tx, Package_QFP:LQFP-32_7x7mm_P0.8mm, F.Cu at (168.1, 96.8)
- added U10: TLP291, Package_SO:SOIC-4_4.55x2.6mm_P1.27mm, F.Cu at (59.4, 85.4)
- added U11: TLP291, Package_SO:SOIC-4_4.55x2.6mm_P1.27mm, F.Cu at (59.4, 89.5)
- added U12: TLP291, Package_SO:SOIC-4_4.55x2.6mm_P1.27mm, F.Cu at (59.4, 93.7)
- added U13: TLP291, Package_SO:SOIC-4_4.55x2.6mm_P1.27mm, F.Cu at (59.4, 97.8)
- added U3: NJM78L12SU3, Package_TO_SOT_SMD:TO-252-2, F.Cu at (73.3, 115.3)
- added U4: TLP291, Package_SO:SOIC-4_4.55x2.6mm_P1.27mm, F.Cu at (59.4, 60.5)
- added U5: TLP291, Package_SO:SOIC-4_4.55x2.6mm_P1.27mm, F.Cu at (59.4, 64.6)
- added U6: TLP291, Package_SO:SOIC-4_4.55x2.6mm_P1.27mm, F.Cu at (59.4, 68.8)
- added U7: TLP291, Package_SO:SOIC-4_4.55x2.6mm_P1.27mm, F.Cu at (59.4, 72.9)
- added U8: TLP291, Package_SO:SOIC-4_4.55x2.6mm_P1.27mm, F.Cu at (59.4, 77.1)
- added U9: TLP291, Package_SO:SOIC-4_4.55x2.6mm_P1.27mm, F.Cu at (59.4, 81.2)

Commit message: update
Parts:
- removed ? (x2): , 
- removed the J1 at (124.7, 69.5)
- removed the J1 at (164.5, 82.7)
- removed the J2 at (113.1, 69.4)
- removed the J2 at (178.0, 82.7)
- removed J4, J5: Conn_01x02, Connector_JST:JST_XH_S2B-XH-A_1x02_P2.50mm_Horizontal
- removed Q1, Q2: AO3400A, Package_TO_SOT_SMD:SOT-23
- removed R15, R16, R26, R27: R, Resistor_SMD:R_0603_1608Metric_Pad0.98x0.95mm_HandSolder
- removed U10, U11, U12, U13, U6, U7, U8, U9: TLP291, Package_SO:SOIC-4_4.55x2.6mm_P1.27mm
- added C11: 4.7u, Capacitor_SMD:C_0603_1608Metric_Pad1.08x0.95mm_HandSolder, F.Cu at (160.6, 94.0)
- added C12: 0.1u, Capacitor_SMD:C_0603_1608Metric_Pad1.08x0.95mm_HandSolder, F.Cu at (138.0, 91.6)
- added C13: 0.1u, Capacitor_SMD:C_0603_1608Metric_Pad1.08x0.95mm_HandSolder, F.Cu at (163.5, 91.8)
- added C9: 0.1u, Capacitor_SMD:C_0603_1608Metric_Pad1.08x0.95mm_HandSolder, F.Cu at (159.0, 94.0)
- added D1: D, 0-Myparts:SS2040FL, F.Cu at (166.9, 94.8)
- added G***: LOGO, 0-Myparts:smallshcale, F.Cu at (106.9, 91.0)
- added IC1: TJA1441AT_0Z, 0-Myparts:SOIC127P600X175-8N, F.Cu at (163.2, 88.0)
- added J1: Conn_01x04, Connector_JST:JST_XH_S4B-XH-A_1x04_P2.50mm_Horizontal, B.Cu at (158.0, 82.6)
- added J16: Conn_01x04, Connector_PinHeader_2.54mm:PinHeader_1x04_P2.54mm_Vertical, F.Cu at (153.1, 82.4)
- added J17: Conn_01x01_Pin, 0-Myparts:ねじ端子(縦), F.Cu at (124.7, 69.2)
- added J18: Conn_01x01_Pin, 0-Myparts:ねじ端子(縦), F.Cu at (113.1, 69.2)
- added J2: Conn_01x04, Connector_JST:JST_XH_S4B-XH-A_1x04_P2.50mm_Horizontal, B.Cu at (171.5, 82.6)
- added JP1: Jumper_2_Bridged, Connector_PinHeader_2.54mm:PinHeader_1x02_P2.54mm_Vertical, F.Cu at (174.8, 87.3)
- added R42: 10k, Resistor_SMD:R_0603_1608Metric, F.Cu at (141.8, 91.6)
- added R43: 120, Resistor_SMD:R_0603_1608Metric, F.Cu at (168.0, 87.8)
- added SW1: SW_Push, 0-Myparts:TVAF06, F.Cu at (137.2, 96.1)
- added SW2: SW_Push, 0-Myparts:TVAF06, F.Cu at (141.0, 96.0)
- added U2: ADP3338AKCZ-3.3, 0-Myparts:SOT230P700X180-4N, F.Cu at (172.0, 93.4)
- J13, J14, R10, R11, R12, R13, R14, R7, R8, R9: moved to B.Cu
- U4, U5: value TLP291 -> TLP291-4; footprint Package_SO:SOIC-4_4.55x2.6mm_P1.27mm -> Package_SO:SOIC-16_4.55x10.3mm_P1.27mm
- moved R6 157.5 mm to (175.5, 98.8), turned to -90 degrees
- moved R5 156.6 mm to (175.5, 107.4), turned to -90 degrees
- moved C3 150.3 mm to (169.2, 99.4), turned to 180 degrees
- moved J12 148.4 mm to (175.1, 118.0)
- moved R24 145.0 mm to (172.6, 112.9), turned to 180 degrees
- moved C2 144.7 mm to (163.5, 94.8), turned to 180 degrees
- moved J13 141.6 mm to (180.5, 95.4), turned to -90 degrees
- moved R34 140.8 mm to (172.6, 111.2)
- moved R14 140.6 mm to (163.1, 97.8), turned to 90 degrees
- moved R13 137.8 mm to (160.5, 97.8), turned to 90 degrees
- moved R23 136.5 mm to (164.1, 112.9), turned to 180 degrees
- moved J8 135.1 mm to (157.9, 118.0)
- moved R12 135.1 mm to (158.0, 97.8), turned to 90 degrees
- moved J3 132.9 mm to (140.6, 118.0)
- moved J14 132.9 mm to (180.5, 104.0), turned to -90 degrees
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Connections:
- C5 pad 1: unconnected-(C5-Pad1) -> +24V
- J13 pad 1: +24V -> +3.3V
- J14 pad 1: +24V -> +3.3V
- J3 pad 2: O1 -> O6
- R5 pad 1: SN1 -> SW2
- R6 pad 1: SN2 -> SW1
- U1 pad 14: SW1 -> SW2
- U1 pad 15: SW2 -> SW1
- U1 pad 2: SN1 -> unconnected-(U1-PF0-Pad2)
- U1 pad 3: SN2 -> unconnected-(U1-PF1-Pad3)
- U1 pad 31: unconnected-(U1-BOOT0-Pad31) -> BOOT
- U1 pad 4: unconnected-(U1-NRST-Pad4) -> NRST
- U4 pad 1: SN1 -> SN6
- U4 pad 3: Net-(R15-Pad2) -> SN5
- U4 pad 4: +8V -> GND
- U5 pad 1: SN2 -> SN10
- U5 pad 3: Net-(R16-Pad2) -> SN9
- U5 pad 4: +8V -> GND
Routing:
- net +24V: track 0.00 -> 137.8 mm
- net +3.3V: track 0.00 -> 121.9 mm, vias 0 -> 4
- net +8V: track 0.00 -> 72.8 mm
- net VCC: track 0.00 -> 53.4 mm, vias 0 -> 2
- net Net-(R17-Pad2): track 0.00 -> 35.2 mm
- net CANH: track 0.00 -> 32.5 mm
- net Net-(R18-Pad2): track 0.00 -> 30.0 mm
- net SW2: track 0.00 -> 29.4 mm
- net SW1: track 0.00 -> 28.1 mm
- net CANL: track 0.00 -> 26.5 mm, vias 0 -> 1
- net Net-(R19-Pad2): track 0.00 -> 23.2 mm
- net LED7: track 0.00 -> 18.9 mm
- net LED1: track 0.00 -> 18.2 mm
- net Net-(R20-Pad2): track 0.00 -> 17.4 mm
- net NRST: track 0.00 -> 17.0 mm
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- added copper zone on B.Cu, net GND
- added copper zone on F.Cu, net GND
- added copper zone on B.Cu, net GNDPWR
- added copper zone on F.Cu, net GNDPWR

Commit message: update
Parts:
- moved J13 0.41 mm to (180.1, 95.4)
- moved J14 0.41 mm to (180.1, 104.0)
Routing:
- net +24V: track 137.8 -> 146.8 mm
- net GNDPWR: vias 0 -> 64
